Commit message: lardemua/larcc#25 solving gripper path issues.

File: ur_description/urdf/inc/ur_macro.xacro (robot description, xacro)
@@ -309,11 +309,11 @@
     </joint>
     <!-- ROS-Industrial 'tool0' frame: all-zeros tool frame -->
-    <link name="${prefix}tool0"/>
-    <joint name="${prefix}flange-tool0" type="fixed">
-      <!-- default toolframe: X+ left, Y+ up, Z+ front -->
-      <origin xyz="0 0 0" rpy="${pi/2.0} 0 ${pi/2.0}"/>
-      <parent link="${prefix}flange"/>
-      <child link="${prefix}tool0"/>
-    </joint>
+<!--    <link name="${prefix}tool0"/>-->
+<!--    <joint name="${prefix}flange-tool0" type="fixed">-->
+<!--      &lt;!&ndash; default toolframe: X+ left, Y+ up, Z+ front &ndash;&gt;-->
+<!--      <origin xyz="0 0 0" rpy="${pi/2.0} 0 ${pi/2.0}"/>-->
+<!--      <parent link="${prefix}flange"/>-->
+<!--      <child link="${prefix}tool0"/>-->
+<!--    </joint>-->
   </xacro:macro>
 </robot>

Commit message: lardemua/larcc#23 Working with use_sim_time = true (when recording)

File: ur_description/urdf/inc/ur_macro.xacro (robot description, xacro)
@@ -309,11 +309,11 @@
     </joint>
     <!-- ROS-Industrial 'tool0' frame: all-zeros tool frame -->
-<!--    <link name="${prefix}tool0"/>-->
-<!--    <joint name="${prefix}flange-tool0" type="fixed">-->
-<!--      &lt;!&ndash; default toolframe: X+ left, Y+ up, Z+ front &ndash;&gt;-->
-<!--      <origin xyz="0 0 0" rpy="${pi/2.0} 0 ${pi/2.0}"/>-->
-<!--      <parent link="${prefix}flange"/>-->
-<!--      <child link="${prefix}tool0"/>-->
-<!--    </joint>-->
+    <link name="${prefix}tool0"/>
+    <joint name="${prefix}flange-tool0" type="fixed">
+      <!-- default toolframe: X+ left, Y+ up, Z+ front -->
+      <origin xyz="0 0 0" rpy="${pi/2.0} 0 ${pi/2.0}"/>
+      <parent link="${prefix}flange"/>
+      <child link="${prefix}tool0"/>
+    </joint>
   </xacro:macro>
 </robot>
